Commit message: split "scout" and "scout with bumper" models; made cmake build xacro

File: models/bunker/model.xacro (robot description, xacro)
@@ -2,9 +2,9 @@
 <sdf version="1.10" xmlns:xacro="http://ros.org/wiki/xacro">
 <model name='bunker' canonical_link='base_link'>
-  <xacro:property name="update_rate_odom"      value="1"/>
-  <xacro:property name="update_rate_imu"       value="1"/>
-  <xacro:property name="update_rate_pose"      value="1"/>
-  <xacro:property name="linear_speed"          value="1"/>
-  <xacro:property name="angular_speed"         value="1"/>
+  <xacro:property name="update_rate_odom" value="1" />
+  <xacro:property name="update_rate_imu" value="1" />
+  <xacro:property name="update_rate_pose" value="1" />
+  <xacro:property name="linear_speed" value="1" />
+  <xacro:property name="angular_speed" value="1" />
   <!-- base_link -->
   <link name='base_link'>
@@ -104,5 +104,5 @@
     </link>
     <joint name="wheel${N}_joint" type="revolute">
-      <pose relative_to='wheel${N}_Link'/>
+      <pose relative_to='wheel${N}_Link' />
       <parent>base_link</parent>
       <child>wheel${N}_Link</child>
@@ -116,24 +116,217 @@
     </joint>
   </xacro:macro>
-  <xacro:wheel N='1'   R='0.05'  W='0.15' P='-0.075' m='2' X='0.44403'  Y='0.3495'  Z='-0.12853' r='1.5708' p='0.0' y='-3.1416'/>
-  <xacro:wheel N='1.1' R='0.04'  W='0.15' P='-0.075' m='1' X='0.37551'  Y='0.3495'  Z='-0.22305' r='1.5708' p='0.0' y='-3.1416'/>
-  <xacro:wheel N='1.2' R='0.05'  W='0.15' P='-0.075' m='1' X='0.29039'  Y='0.3495'  Z='-0.28104' r='1.5708' p='0.0' y='-3.1416'/>
-  <xacro:wheel N='1.3' R='0.05'  W='0.15' P='-0.075' m='1' X='0.29603'  Y='0.3495'  Z='-0.087'   r='1.5708' p='0.0' y='-3.1416'/>
-  <xacro:wheel N='2'   R='0.05'  W='0.15' P='0.075'  m='2' X='0.44403'  Y='-0.3495' Z='-0.12853' r='1.5708' p='0.0' y='-3.1416'/>
-  <xacro:wheel N='2.1' R='0.04'  W='0.15' P='0.075'  m='1' X='0.37551'  Y='-0.3495' Z='-0.22305' r='1.5708' p='0.0' y='-3.1416'/>
-  <xacro:wheel N='2.2' R='0.05'  W='0.15' P='0.075'  m='1' X='0.29039'  Y='-0.3495' Z='-0.28104' r='1.5708' p='0.0' y='-3.1416'/>
-  <xacro:wheel N='2.3' R='0.05'  W='0.15' P='0.075'  m='1' X='0.29603'  Y='-0.3495' Z='-0.087'   r='1.5708' p='0.0' y='-3.1416'/>
-  <xacro:wheel N='3'   R='0.075' W='0.15' P='-0.025' m='8' X='-0.38871' Y='0.295'   Z='-0.19381' r='1.5708' p='0.0' y='-3.1416'/>
-  <xacro:wheel N='3.1' R='0.05'  W='0.15' P='-0.075' m='1' X='-0.23111' Y='0.3495'  Z='-0.27671' r='1.5708' p='0.0' y='-3.1416'/>
-  <xacro:wheel N='3.2' R='0.05'  W='0.15' P='-0.075' m='1' X='0.043885' Y='0.3495'  Z='-0.27671' r='1.5708' p='0.0' y='-3.1416'/>
-  <xacro:wheel N='3.3' R='0.05'  W='0.15' P='-0.075' m='1' X='-0.28597' Y='0.3495'  Z='-0.087'   r='1.5708' p='0.0' y='-3.1416'/>
-  <xacro:wheel N='4'   R='0.075' W='0.15' P='0.025'  m='8' X='-0.38871' Y='-0.295'  Z='-0.19381' r='1.5708' p='0.0' y='-3.1416'/>
-  <xacro:wheel N='4.1' R='0.05'  W='0.15' P='0.075'  m='1' X='-0.23111' Y='-0.3495' Z='-0.27671' r='1.5708' p='0.0' y='-3.1416'/>
-  <xacro:wheel N='4.2' R='0.05'  W='0.15' P='0.075'  m='1' X='0.043885' Y='-0.3495' Z='-0.27671' r='1.5708' p='0.0' y='-3.1416'/>
-  <xacro:wheel N='4.3' R='0.05'  W='0.15' P='0.075'  m='1' X='-0.28597' Y='-0.3495' Z='-0.087'   r='1.5708' p='0.0' y='-3.1416'/>
+  <xacro:wheel
+            N='1'
+            R='0.05'
+            W='0.15'
+            P='-0.075'
+            m='2'
+            X='0.44403'
+            Y='0.3495'
+            Z='-0.12853'
+            r='1.5708'
+            p='0.0'
+            y='-3.1416'
+        />
+  <xacro:wheel
+            N='1.1'
+            R='0.04'
+            W='0.15'
+            P='-0.075'
+            m='1'
+            X='0.37551'
+            Y='0.3495'
+            Z='-0.22305'
+            r='1.5708'
+            p='0.0'
+            y='-3.1416'
+        />
+  <xacro:wheel
+            N='1.2'
+            R='0.05'
+            W='0.15'
+            P='-0.075'
+            m='1'
+            X='0.29039'
+            Y='0.3495'
+            Z='-0.28104'
+            r='1.5708'
+            p='0.0'
+            y='-3.1416'
+        />
+  <xacro:wheel
+            N='1.3'
+            R='0.05'
+            W='0.15'
+            P='-0.075'
+            m='1'
+            X='0.29603'
+            Y='0.3495'
+            Z='-0.087'
+            r='1.5708'
+            p='0.0'
+            y='-3.1416'
+        />
+  <xacro:wheel
+            N='2'
+            R='0.05'
+            W='0.15'
+            P='0.075'
+            m='2'
+            X='0.44403'
+            Y='-0.3495'
+            Z='-0.12853'
+            r='1.5708'
+            p='0.0'
+            y='-3.1416'
+        />
+  <xacro:wheel
+            N='2.1'
+            R='0.04'
+            W='0.15'
+            P='0.075'
+            m='1'
+            X='0.37551'
+            Y='-0.3495'
+            Z='-0.22305'
+            r='1.5708'
+            p='0.0'
+            y='-3.1416'
+        />
+  <xacro:wheel
+            N='2.2'
+            R='0.05'
+            W='0.15'
+            P='0.075'
+            m='1'
+            X='0.29039'
+            Y='-0.3495'
+            Z='-0.28104'
+            r='1.5708'
+            p='0.0'
+            y='-3.1416'
+        />
+  <xacro:wheel
+            N='2.3'
+            R='0.05'
+            W='0.15'
+            P='0.075'
+            m='1'
+            X='0.29603'
+            Y='-0.3495'
+            Z='-0.087'
+            r='1.5708'
+            p='0.0'
+            y='-3.1416'
+        />
+  <xacro:wheel
+            N='3'
+            R='0.075'
+            W='0.15'
+            P='-0.025'
+            m='8'
+            X='-0.38871'
+            Y='0.295'
+            Z='-0.19381'
+            r='1.5708'
+            p='0.0'
+            y='-3.1416'
+        />
+  <xacro:wheel
+            N='3.1'
+            R='0.05'
+            W='0.15'
+            P='-0.075'
+            m='1'
+            X='-0.23111'
+            Y='0.3495'
+            Z='-0.27671'
+            r='1.5708'
+            p='0.0'
+            y='-3.1416'
+        />
+  <xacro:wheel
+            N='3.2'
+            R='0.05'
+            W='0.15'
+            P='-0.075'
+            m='1'
+            X='0.043885'
+            Y='0.3495'
+            Z='-0.27671'
+            r='1.5708'
+            p='0.0'
+            y='-3.1416'
+        />
+  <xacro:wheel
+            N='3.3'
+            R='0.05'
+            W='0.15'
+            P='-0.075'
+            m='1'
+            X='-0.28597'
+            Y='0.3495'
+            Z='-0.087'
+            r='1.5708'
+            p='0.0'
+            y='-3.1416'
+        />
+  <xacro:wheel
+            N='4'
+            R='0.075'
+            W='0.15'
+            P='0.025'
+            m='8'
+            X='-0.38871'
+            Y='-0.295'
+            Z='-0.19381'
+            r='1.5708'
+            p='0.0'
+            y='-3.1416'
+        />
+  <xacro:wheel
+            N='4.1'
+            R='0.05'
+            W='0.15'
+            P='0.075'
+            m='1'
+            X='-0.23111'
+            Y='-0.3495'
+            Z='-0.27671'
+            r='1.5708'
+            p='0.0'
+            y='-3.1416'
+        />
+  <xacro:wheel
+            N='4.2'
+            R='0.05'
+            W='0.15'
+            P='0.075'
+            m='1'
+            X='0.043885'
+            Y='-0.3495'
+            Z='-0.27671'
+            r='1.5708'
+            p='0.0'
+            y='-3.1416'
+        />
+  <xacro:wheel
+            N='4.3'
+            R='0.05'
+            W='0.15'
+            P='0.075'
+            m='1'
+            X='-0.28597'
+            Y='-0.3495'
+            Z='-0.087'
+            r='1.5708'
+            p='0.0'
+            y='-3.1416'
+        />
   <!-- plugins -->
   <plugin
-    filename="gz-sim-diff-drive-system"
-    name="gz::sim::systems::DiffDrive">
+            filename="gz-sim-diff-drive-system"
+            name="gz::sim::systems::DiffDrive"
+        >
     <left_joint>wheel1_joint</left_joint>
     <left_joint>wheel1.1_joint</left_joint>
@@ -157,6 +350,7 @@
   <xacro:macro name="keymap" params="D L A">
     <plugin
-      filename="gz-sim-triggered-publisher-system"
-      name="gz::sim::systems::TriggeredPublisher">
+                filename="gz-sim-triggered-publisher-system"
+                name="gz::sim::systems::TriggeredPublisher"
+            >
       <input type="gz.msgs.Int32" topic="/keyboard/keypress">
         <match field="data">${D}</match>
@@ -168,16 +362,17 @@
   </xacro:macro>
   <!-- FrontArrowKey: drive frontward -->
-  <xacro:keymap D='16777235' L='${linear_speed}'    A='0.0'/>
+  <xacro:keymap D='16777235' L='${linear_speed}' A='0.0' />
   <!-- BackArrowKey: drive backward -->
-  <xacro:keymap D='16777237' L='${(-linear_speed)}' A='0.0'/>
+  <xacro:keymap D='16777237' L='${(-linear_speed)}' A='0.0' />
   <!-- LeftArrowKey: turn left -->
-  <xacro:keymap D='16777234' L='0.0'                A='${angular_speed}'/>
+  <xacro:keymap D='16777234' L='0.0' A='${angular_speed}' />
   <!-- RightArrowKey: turn right -->
-  <xacro:keymap D='16777236' L='0.0'                A='${(-angular_speed)}'/>
+  <xacro:keymap D='16777236' L='0.0' A='${(-angular_speed)}' />
   <!-- s: stop -->
-  <xacro:keymap D='83'       L='0.0'                A='0.0'/>
+  <xacro:keymap D='83' L='0.0' A='0.0' />
   <plugin
-    filename="gz-sim-pose-publisher-system"
-    name="gz::sim::systems::PosePublisher">
+            filename="gz-sim-pose-publisher-system"
+            name="gz::sim::systems::PosePublisher"
+        >
     <publish_link_pose>False</publish_link_pose>
     <publish_visual_pose>False</publish_visual_pose>
@@ -191,7 +386,5 @@
     <static_update_frequency>${update_rate_pose}</static_update_frequency>
   </plugin>
-  <plugin
-    filename="gz-sim-imu-system"
-    name="gz::sim::systems::Imu">
+  <plugin filename="gz-sim-imu-system" name="gz::sim::systems::Imu">
   </plugin>
 </model>

File: models/scout/model.xacro (robot description, xacro)
@@ -2,10 +2,9 @@
 <sdf version="1.10" xmlns:xacro="http://ros.org/wiki/xacro">
 <model name='scout' canonical_link='chassis'>
-  <xacro:property name="update_rate_odom"      value="1"/>
-  <xacro:property name="update_rate_imu"       value="1"/>
-  <xacro:property name="update_rate_pose"      value="3"/>
-  <xacro:property name="update_rate_force_bar" value="1000"/>
-  <xacro:property name="linear_speed"          value="0.5"/>
-  <xacro:property name="angular_speed"         value="0.5"/>
+  <xacro:property name="update_rate_odom" value="1" />
+  <xacro:property name="update_rate_imu" value="1" />
+  <xacro:property name="update_rate_pose" value="3" />
+  <xacro:property name="linear_speed" value="0.5" />
+  <xacro:property name="angular_speed" value="0.5" />
   <!-- base_link -->
   <link name='chassis'>
@@ -34,8 +33,8 @@
   </link>
   <!-- wheels -->
-  <xacro:property name="wheel_radius"     value="0.16"/>
-  <xacro:property name="wheel_width"      value="0.11"/>
-  <xacro:property name="wheel_base"       value="0.498"/>
-  <xacro:property name="wheel_separation" value="0.58306"/>
+  <xacro:property name="wheel_radius" value="0.16" />
+  <xacro:property name="wheel_width" value="0.11" />
+  <xacro:property name="wheel_base" value="0.498" />
+  <xacro:property name="wheel_separation" value="0.58306" />
   <xacro:macro name="wheel" params="N T X Y Z r p y">
     <link name='${N}_wheel'>
@@ -50,5 +49,7 @@
       </visual>
       <collision name='collision'>
-        <pose relative_to="chassis">${X} ${Y} ${Z} ${((pi/2)-r)} ${p} ${y}</pose>
+        <pose
+                        relative_to="chassis"
+                    >${X} ${Y} ${Z} ${((pi/2)-r)} ${p} ${y}</pose>
         <geometry>
           <cylinder>
@@ -60,5 +61,5 @@
     </link>
     <joint name='${N}_wheel_joint' type='revolute'>
-      <pose relative_to='${N}_wheel'/>
+      <pose relative_to='${N}_wheel' />
       <parent>chassis</parent>
       <child>${N}_wheel</child>
@@ -72,81 +73,49 @@
     </joint>
   </xacro:macro>
-  <xacro:wheel N='front_left'  T='2' X='${(wheel_base/2)}'  Y='${(wheel_separation/2)}'  Z='-0.0702' r='0.0'   p='0.0' y='0.0'/>
-  <xacro:wheel N='front_right' T='1' X='${(wheel_base/2)}'  Y='${(-wheel_separation/2)}' Z='-0.0702' r='${pi}' p='0.0' y='0.0'/>
-  <xacro:wheel N='back_left'   T='1' X='${(-wheel_base/2)}' Y='${(wheel_separation/2)}'  Z='-0.0702' r='0.0'   p='0.0' y='0.0'/>
-  <xacro:wheel N='back_right'  T='2' X='${(-wheel_base/2)}' Y='${(-wheel_separation/2)}' Z='-0.0702' r='${pi}' p='0.0' y='0.0'/>
-  <!-- visual connection -->
-  <xacro:macro name="force_bar_material">
-    <material>
-      <ambient>0.25 0.25 0.25 1.0</ambient>
-      <diffuse>0.25 0.25 0.25 1.0</diffuse>
-      <specular>0.25 0.25 0.25 1.0</specular>
-    </material>
-  </xacro:macro>
-  <xacro:macro name="force_bar_connection_visual" params="N X Y Z r p y L W H">
-    <visual name='force_bar_connection_visual_${N}'>
-      <pose relative_to="chassis">${X} ${Y} ${Z} ${r} ${p} ${y}</pose>
-      <geometry>
-        <box>
-          <size>${L} ${W} ${H}</size>
-        </box>
-      </geometry>
-      <xacro:force_bar_material/>
-    </visual>
-  </xacro:macro>
-  <link name='force_bar_connection_visual'>
-    <xacro:force_bar_connection_visual N='center_bar_left'  X='0.4'    Y='0.04'   Z='0' r='0' p='0' y='0'        L='0.2'   W='0.025' H='0.025'/>
-    <xacro:force_bar_connection_visual N='center_bar_right' X='0.4'    Y='-0.04'  Z='0' r='0' p='0' y='0'        L='0.2'   W='0.025' H='0.025'/>
-    <xacro:force_bar_connection_visual N='front_bar_top'    X='0.4875' Y='0'      Z='0' r='0' p='0' y='0'        L='0.025' W='0.41'  H='0.025'/>
-    <xacro:force_bar_connection_visual N='front_bar_left'   X='0.4575' Y='0.265'  Z='0' r='0' p='0' y='0.43633'  L='0.025' W='0.15'  H='0.025'/>
-    <xacro:force_bar_connection_visual N='front_bar_right'  X='0.4575' Y='-0.265' Z='0' r='0' p='0' y='-0.43633' L='0.025' W='0.15'  H='0.025'/>
-  </link>
-  <joint name='force_bar_connection_visual_joint' type='fixed'>
-    <pose relative_to='force_bar_connection_visual'/>
-    <parent>chassis</parent>
-    <child>force_bar_connection_visual</child>
-  </joint>
-  <!-- sensor bar -->
-  <xacro:macro name="force_bar_segment" params="P X Y Z r p y L W H">
-    <link name='force_bar_P${P}_link'>
-      <pose relative_to="chassis">${X} ${Y} ${Z} ${r} ${p} ${y}</pose>
-      <inertial auto="true">
-        <mass>1</mass>
-      </inertial>
-      <visual name='visual'>
-        <geometry>
-          <box>
-            <size>${L} ${W} ${H}</size>
-          </box>
-        </geometry>
-        <xacro:force_bar_material/>
-      </visual>
-      <collision name='collision'>
-        <geometry>
-          <box>
-            <size>${L} ${W} ${H}</size>
-          </box>
-        </geometry>
-      </collision>
-    </link>
-    <joint name='force_bar_P${P}_joint' type='fixed'>
-      <pose relative_to='force_bar_P${P}_link'/>
-      <parent>chassis</parent>
-      <child>force_bar_P${P}_link</child>
-      <sensor name='force_bar_P${P}_sensor' type='force_torque'>
-        <always_on>true</always_on>
-        <update_rate>${update_rate_force_bar}</update_rate>
-        <visualize>true</visualize>
-        <topic>/scout/force_bar/segment_${P}</topic>
-      </sensor>
-    </joint>
-  </xacro:macro>
-  <xacro:force_bar_segment P='0' X='0.466' Y='0.28'  Z='0.0' r='${pi/2}' p='0.0' y='0.43633'  L='0.005' W='0.15' H='0.14'/>
-  <xacro:force_bar_segment P='1' X='0.5'   Y='0.14'  Z='0.0' r='${pi/2}' p='0.0' y='0.0'      L='0.005' W='0.15' H='0.13'/>
-  <xacro:force_bar_segment P='2' X='0.5'   Y='0.0'   Z='0.0' r='${pi/2}' p='0.0' y='0.0'      L='0.005' W='0.15' H='0.13'/>
-  <xacro:force_bar_segment P='3' X='0.5'   Y='-0.14' Z='0.0' r='${pi/2}' p='0.0' y='0.0'      L='0.005' W='0.15' H='0.13'/>
-  <xacro:force_bar_segment P='4' X='0.466' Y='-0.28' Z='0.0' r='${pi/2}' p='0.0' y='-0.43633' L='0.005' W='0.15' H='0.14'/>
+  <xacro:wheel
+            N='front_left'
+            T='2'
+            X='${(wheel_base/2)}'
+            Y='${(wheel_separation/2)}'
+            Z='-0.0702'
+            r='0.0'
+            p='0.0'
+            y='0.0'
+        />
+  <xacro:wheel
+            N='front_right'
+            T='1'
+            X='${(wheel_base/2)}'
+            Y='${(-wheel_separation/2)}'
+            Z='-0.0702'
+            r='${pi}'
+            p='0.0'
+            y='0.0'
+        />
+  <xacro:wheel
+            N='back_left'
+            T='1'
+            X='${(-wheel_base/2)}'
+            Y='${(wheel_separation/2)}'
+            Z='-0.0702'
+            r='0.0'
+            p='0.0'
+            y='0.0'
+        />
+  <xacro:wheel
+            N='back_right'
+            T='2'
+            X='${(-wheel_base/2)}'
+            Y='${(-wheel_separation/2)}'
+            Z='-0.0702'
+            r='${pi}'
+            p='0.0'
+            y='0.0'
+        />
   <!-- plugins -->
-  <plugin filename="gz-sim-diff-drive-system" name="gz::sim::systems::DiffDrive">
+  <plugin
+            filename="gz-sim-diff-drive-system"
+            name="gz::sim::systems::DiffDrive"
+        >
     <!-- wheels -->
     <left_joint>front_left_wheel_joint</left_joint>
@@ -157,24 +126,20 @@
     <wheel_separation>${wheel_separation}</wheel_separation>
     <wheel_radius>${wheel_radius}</wheel_radius>
-    <!-- limits -->
-    <!-- <max_linear_acceleration>0.1</max_linear_acceleration> -->
     <!-- input -->
     <topic>/cmd_vel</topic>
     <!-- output -->
     <odom_publish_frequency>${update_rate_odom}</odom_publish_frequency>
-    <!-- <odom_topic>/nav/odom</odom_topic> -->
-    <!-- <tf_topic>/tf</tf_topic> -->
-    <!-- <frame_id>odom</frame_id> -->
-    <!-- <child_frame_id>base_link</child_frame_id> -->
   </plugin>
   <plugin
-      filename="gz-sim-joint-state-publisher-system"
-      name="gz::sim::systems::JointStatePublisher">
+            filename="gz-sim-joint-state-publisher-system"
+            name="gz::sim::systems::JointStatePublisher"
+        >
       <topic>joint_states</topic>
   </plugin>
   <xacro:macro name="keymap" params="D L A">
     <plugin
-      filename="gz-sim-triggered-publisher-system"
-      name="gz::sim::systems::TriggeredPublisher">
+                filename="gz-sim-triggered-publisher-system"
+                name="gz::sim::systems::TriggeredPublisher"
+            >
       <input type="gz.msgs.Int32" topic="/keyboard/keypress">
         <match field="data">${D}</match>
@@ -186,16 +151,17 @@
   </xacro:macro>
   <!-- FrontArrowKey: drive frontward -->
-  <xacro:keymap D='16777235' L='${linear_speed}'    A='0.0'/>
+  <xacro:keymap D='16777235' L='${linear_speed}' A='0.0' />
   <!-- BackArrowKey: drive backward -->
-  <xacro:keymap D='16777237' L='${(-linear_speed)}' A='0.0'/>
+  <xacro:keymap D='16777237' L='${(-linear_speed)}' A='0.0' />
   <!-- LeftArrowKey: turn left -->
-  <xacro:keymap D='16777234' L='0.0'                A='${angular_speed}'/>
+  <xacro:keymap D='16777234' L='0.0' A='${angular_speed}' />
   <!-- RightArrowKey: turn right -->
-  <xacro:keymap D='16777236' L='0.0'                A='${(-angular_speed)}'/>
+  <xacro:keymap D='16777236' L='0.0' A='${(-angular_speed)}' />
   <!-- s: stop -->
-  <xacro:keymap D='83'       L='0.0'                A='0.0'/>
+  <xacro:keymap D='83' L='0.0' A='0.0' />
   <plugin
-    filename="gz-sim-pose-publisher-system"
-    name="gz::sim::systems::PosePublisher">
+            filename="gz-sim-pose-publisher-system"
+            name="gz::sim::systems::PosePublisher"
+        >
     <publish_link_pose>False</publish_link_pose>
     <publish_visual_pose>False</publish_visual_pose>
@@ -209,11 +175,5 @@
     <static_update_frequency>${update_rate_pose}</static_update_frequency>
   </plugin>
-  <plugin
-    filename="gz-sim-imu-system"
-    name="gz::sim::systems::Imu">
-  </plugin>
-  <plugin
-    filename="gz-sim-forcetorque-system"
-    name="gz::sim::systems::ForceTorque">
+  <plugin filename="gz-sim-imu-system" name="gz::sim::systems::Imu">
   </plugin>
 </model>
